File: ETC/ETC.kicad_pcb (KiCad board)
At the start: 2 copper layers, 36 parts, among them P1 DTM1312PC12PDR008, U1 NUCLEO-F446RE, U2 MCP6004, U3 LM7805_TO220, U4 LM7809_TO220, U5 ISO1050DUB, U6 ISO1050DUB, U7 SN74AHC14N

Commit message: Update ETC.kicad_pcb
Parts:
- added C14: 100 nF, Capacitor_SMD:C_0805_2012Metric_Pad1.18x1.45mm_HandSolder, F.Cu at (88.0, 52.8)
- added C15: 100 nF, Capacitor_SMD:C_0805_2012Metric_Pad1.18x1.45mm_HandSolder, F.Cu at (94.5, 102.0)
- added R16: 1kΩ, Resistor_SMD:R_0805_2012Metric_Pad1.20x1.40mm_HandSolder, F.Cu at (108.5, 46.3)
- added R17: 200kΩ, Resistor_SMD:R_0805_2012Metric_Pad1.20x1.40mm_HandSolder, F.Cu at (113.0, 49.3)
- added R18: 1kΩ, Resistor_SMD:R_0805_2012Metric_Pad1.20x1.40mm_HandSolder, F.Cu at (121.5, 81.3)
- added R19: 200kΩ, Resistor_SMD:R_0805_2012Metric_Pad1.20x1.40mm_HandSolder, F.Cu at (103.0, 102.0)
- moved C13 121.3 mm to (100.5, 125.0), turned to 90 degrees
- moved C11 115.1 mm to (93.0, 125.0), turned to 90 degrees
- moved R15 94.1 mm to (138.5, 128.5)
- moved C1 88.6 mm to (146.5, 129.0)
- moved C3 76.2 mm to (146.5, 123.5)
- moved U3 75.4 mm to (134.5, 115.1)
- moved U4 63.3 mm to (65.5, 91.3), turned to 90 degrees
- moved U5 60.8 mm to (129.0, 59.3), turned to 180 degrees
- moved U6 55.7 mm to (130.5, 77.8)
- moved C4 53.8 mm to (73.0, 87.8), turned to -90 degrees
- moved U7 53.4 mm to (104.5, 63.5), turned to 0 degrees
- moved C12 47.6 mm to (121.5, 76.3), turned to 180 degrees
- moved U2 45.3 mm to (104.8, 88.5), turned to 0 degrees
- moved R13 44.6 mm to (116.5, 56.3), turned to -90 degrees
- moved C10 37.6 mm to (121.5, 70.8), turned to 180 degrees
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
Commit message: Update ETC.kicad_pcb
Parts:
- moved U3 17.4 mm to (131.0, 98.0)
Changed lines of the file:
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@@
 	(footprint "Package_TO_SOT_THT:TO-220-3_Vertical"
 		(layer "F.Cu")
-		(at 134.54 115.055 180)
+		(at 131.04 98 180)
 		(descr "TO-220-3, Vertical, RM 2.54mm, see https://www.vishay.com/docs/66542/to-220-1.pdf")
 		(tags "TO-220-3 Vertical RM 2.54mm")
